Commit message: Configured custom_robot_bringup launch file to launch gz world, custom robot, and SLAM. Renamed robot and its bringup package.

File: src/custom_robot_description/urdf/camera.xacro (robot description, xacro)
@@ -37,4 +37,9 @@
     <gazebo reference="camera_link">
         <sensor name="camera" type="camera">
+            <always_on>1</always_on>
+            <update_rate>20</update_rate>
+            <visualize>true</visualize>
+            <topic>camera/image_raw</topic>
+            <gz_frame_id>camera_link_optical</gz_frame_id>
             <camera>
                 <horizontal_fov>1.3962634</horizontal_fov>
@@ -53,11 +58,6 @@
                     <stddev>0.007</stddev>
                 </noise>
-                <optical_frame_id>camera_link_optical</optical_frame_id>
                 <camera_info_topic>camera/camera_info</camera_info_topic>
             </camera>
-            <always_on>1</always_on>
-            <update_rate>20</update_rate>
-            <visualize>true</visualize>
-            <topic>camera/image_raw</topic>
         </sensor>
     </gazebo>

File: src/custom_robot_description/urdf/custom_robot.urdf.xacro (robot description, xacro)
@@ -5,3 +5,4 @@
     <xacro:include filename="mobile_base_gazebo.xacro" />
     <xacro:include filename="camera.xacro" />
+    <xacro:include filename="lidar.xacro" />
 </robot>

File: src/custom_robot_description/urdf/mobile_base.xacro (robot description, xacro)
@@ -1,10 +1,10 @@
 <?xml version="1.0"?>
 <robot xmlns:xacro="http://www.ros.org/wiki/xacro">
-    <xacro:property name="base_length" value="0.6" />
-    <xacro:property name="base_width" value="0.4" />
-    <xacro:property name="base_height" value="0.2" />
-    <xacro:property name="wheel_radius" value="0.1" />
+    <xacro:property name="base_length" value="0.3" />
+    <xacro:property name="base_width" value="0.2" />
+    <xacro:property name="base_height" value="0.075" />
+    <xacro:property name="wheel_radius" value="0.03" />
     <xacro:property name="wheel_length" value="0.05" />
-    <xacro:property name="sphere_radius" value="0.05" />
+    <xacro:property name="sphere_radius" value="${wheel_radius/2}" />
     <xacro:macro name="wheel_link" params="prefix sign">
         <link name="${prefix}_wheel_link">
@@ -43,5 +43,5 @@
             <origin xyz="0 0 ${base_height / 2.0}" rpy="0 0 0" />
         </collision>
-        <xacro:box_inertia m="5.0" x="${base_length}" y="${base_width}" z="${base_height}"
+        <xacro:box_inertia m="10.0" x="${base_length}" y="${base_width}" z="${base_height}"
                            o_xyz="0 0 ${base_height / 2.0}" o_rpy="0 0 0" />
     </link>
@@ -65,5 +65,5 @@
         <parent link="base_footprint" />
         <child link="base_link" />
-        <origin xyz="0 0 0.1" rpy="0 0 0" />
+        <origin xyz="0 0 ${wheel_radius}" rpy="0 0 0" />
     </joint>
     <joint name="base_caster_wheel_joint" type="fixed">
